File: PCB/HexPad.kicad_pcb (KiCad board)
At the start: 2 copper layers, 62.6 x 65.4 mm, 9 parts, among them J1 Conn_01x04_Socket, SW1 SW_Push, SW2 SW_Push, SW3 SW_Push, SW4 SW_Push, SW5 SW_Push, SW6 SW_Push, SW8 RotaryEncoder_Switch_MP, U1 MOUDLE-SEEEDUINO-XIAO

Commit message: Add files via upload
Parts:
- moved SW3 2.00 mm to (160.0, 99.7)
- moved SW6 2.00 mm to (180.2, 99.7)
- moved SW8 2.00 mm to (191.3, 101.6)
- moved SW2 1.00 mm to (160.0, 80.6)
- moved SW5 1.00 mm to (180.2, 80.6)
Routing:
- net GND: track 177.2 -> 173.2 mm
- net Net-(U1-PA10_A2_D2): track 101.9 -> 105.3 mm
- net Net-(U1-PB09_A7_D7_RX): track 36.6 -> 34.6 mm
- net Net-(U1-PA6_A10_D10_MOSI): track 76.7 -> 74.7 mm
- net Net-(U1-PA02_A0_D0): track 78.5 -> 77.2 mm
- net Net-(U1-PB08_A6_D6_TX): track 19.8 -> 18.8 mm
- net Net-(U1-PA5_A9_D9_MISO): track 50.1 -> 49.1 mm
- net Net-(U1-PA4_A1_D1): track 73.3 -> 72.5 mm
Other:
- board size 62.6 x 65.4 mm -> 62.6 x 63.4 mm

Commit message: Add files via upload
Parts:
- moved J1 4.40 mm to (195.6, 59.3)
- moved SW8 3.50 mm to (191.3, 105.1)
Routing:
- net GND: track 173.2 -> 176.7 mm
- net Net-(U1-PA4_A1_D1): track 72.5 -> 76.0 mm
- net Net-(U1-PA10_A2_D2): track 105.3 -> 102.7 mm
- net Net-(J1-VCC): track 54.0 -> 52.6 mm
- net Net-(U1-PA02_A0_D0): track 77.2 -> 78.2 mm
- net Net-(J1-SDA): track 42.0 -> 41.3 mm
Changed lines of the file:
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@@
 	(footprint "Rotary_Encoder:RotaryEncoder_Alps_EC11E-Switch_Vertical_H20mm"
 		(layer "F.Cu")
-		(at 191.35 101.6)
+		(at 191.35 105.1)
 		(descr "Alps rotary encoder, EC11E... with switch, vertical shaft, http://www.alps.com/prod/info/E/HTML/Encoder/Incremental/EC11/EC11E15204A3.html")
 		(tags "rotary encoder")
@@
 		)
 		(property "Value" "RotaryEncoder_Switch_MP"
-			(at 6.35 11.1 0)
+			(at 6.05 -12 0)
 			(layer "F.Fab")
 			(effects
@@
 	(footprint "Connector_PinSocket_2.54mm:PinSocket_1x04_P2.54mm_Vertical"
 		(layer "F.Cu")
-		(at 195.62 63.7 90)
+		(at 195.62 59.3 90)
 		(descr "Through hole straight socket strip, 1x04, 2.54mm pitch, single row (from Kicad 4.0.7), script generated")
 		(tags "Through hole socket strip THT 1x04 2.54mm single row")
@@
 		)
 		(property "Value" "Conn_01x04_Socket"
-			(at -2.1 10.38 90)
+			(at -5.7 11.08 90)
 			(layer "F.Fab")
 			(effects
@@
 	)
 	(segment
-		(start 198.85 98.5)
-		(end 196.95 98.5)
+		(start 180.22 99.7)
+		(end 186.95 99.7)
 		(width 0.2)
 		(layer "B.Cu")
@@
 	)
 	(segment
-		(start 180.22 99.7)
-		(end 186.95 99.7)
+		(start 196.85 113.2)
+		(end 191.35 107.7)
 		(width 0.2)
 		(layer "B.Cu")
@@
 	)
 	(segment
-		(start 182.4 63.7)
-		(end 180.22 61.52)
+		(start 159.96 99.66)
+		(end 159.96 80.57)
 		(width 0.2)
 		(layer "B.Cu")
@@
 	)
 	(segment
-		(start 159.96 99.66)
-		(end 159.96 80.57)
+		(start 159.96 80.57)
+		(end 159.96 61.48)
 		(width 0.2)
 		(layer "B.Cu")
@@
 	)
 	(segment
-		(start 198.85 109.7)
-		(end 196.95 109.7)
+		(start 186.95 103.2)
+		(end 191.35 107.6)
 		(width 0.2)
 		(layer "B.Cu")
@@
 	)
 	(segment
-		(start 159.96 80.57)
-		(end 159.96 61.48)
+		(start 203.35 107.7)
+		(end 191.35 107.7)
 		(width 0.2)
 		(layer "B.Cu")
@@
 	)
 	(segment
-		(start 203.35 104.1)
-		(end 191.35 104.1)
+		(start 197.05 113.2)
+		(end 198.85 113.2)
+		(width 0.2)
+		(layer "B.Cu")
+		(net 1)
+	)
+	(segment
+		(start 197.05 113.2)
+		(end 196.85 113.2)
 		(width 0.2)
 		(layer "B.Cu")
@@
 	)
 	(segment
-		(start 160 99.7)
-		(end 159.96 99.66)
+		(start 197.05 102)
+		(end 198.85 102)
 		(width 0.2)
 		(layer "B.Cu")
@@
 	)
 	(segment
-		(start 191.35 104.1)
-		(end 186.95 99.7)
+		(start 186.95 99.7)
+		(end 186.95 103.2)
 		(width 0.2)
 		(layer "B.Cu")
@@
 	)
 	(segment
-		(start 180.22 61.52)
-		(end 180.22 80.61)
+		(start 160 99.7)
+		(end 159.96 99.66)
 		(width 0.2)
 		(layer "B.Cu")
@@
 	)
 	(segment
-		(start 196.95 98.5)
-		(end 191.35 104.1)
+		(start 180.22 61.52)
+		(end 180.22 80.61)
 		(width 0.2)
 		(layer "B.Cu")
@@
 	)
 	(segment
-		(start 195.62 63.7)
-		(end 182.4 63.7)
+		(start 159.96 61.48)
+		(end 154.92 56.44)
 		(width 0.2)
 		(layer "B.Cu")
@@
 	)
 	(segment
-		(start 159.96 61.48)
-		(end 154.92 56.44)
+		(start 205.85 105.2)
+		(end 203.35 107.7)
 		(width 0.2)
 		(layer "B.Cu")
@@
 	)
 	(segment
-		(start 205.85 101.6)
-		(end 203.35 104.1)
+		(start 191.35 107.7)
+		(end 197.05 102)
 		(width 0.2)
 		(layer "B.Cu")
@@
 	)
 	(segment
-		(start 196.95 109.7)
-		(end 191.35 104.1)
+		(start 180.22 61.52)
+		(end 193.4 61.52)
 		(width 0.2)
 		(layer "B.Cu")
@@
 	)
 	(segment
-		(start 200.7 63.7)
-		(end 197.12 60.12)
+		(start 193.4 61.52)
+		(end 195.62 59.3)
 		(width 0.2)
 		(layer "B.Cu")
-		(net 2)
+		(net 1)
 	)
 	(segment
-		(start 175.830101 60.12)
+		(start 165.15 66.6)
 		(end 169.350101 66.6)
 		(width 0.2)
@@
 	)
 	(segment
-		(start 197.12 60.12)
-		(end 175.830101 60.12)
+		(start 169.350101 66.6)
+		(end 177.800101 58.15)
 		(width 0.2)
 		(layer "B.Cu")
@@
 	)
 	(segment
-		(start 169.350101 66.6)
-		(end 165.15 66.6)
+		(start 199.55 58.15)
+		(end 200.7 59.3)
 		(width 0.2)
 		(layer "B.Cu")
@@
 	)
 	(segment
-		(start 192.96 58.5)
-		(end 169.6 58.5)
+		(start 177.800101 58.15)
+		(end 199.55 58.15)
+		(width 0.2)
+		(layer "B.Cu")
+		(net 2)
+	)
+	(segment
+		(start 168.3 57.987969)
+		(end 168.462031 58.15)
 		(width 0.2)
 		(layer "F.Cu")
@@
 	)
 	(segment
-		(start 153.59 55.29)
-		(end 149.9 58.98)
+		(start 167.576346 55.29)
+		(end 168.3 56.013654)
 		(width 0.2)
 		(layer "F.Cu")
@@
 	)
 	(segment
-		(start 168.3 57.2)
-		(end 168.3 56.013654)
+		(start 168.462031 58.15)
+		(end 197.01 58.15)
 		(width 0.2)
 		(layer "F.Cu")
@@
 	(segment
 		(start 168.3 56.013654)
-		(end 167.576346 55.29)
+		(end 168.3 57.987969)
 		(width 0.2)
 		(layer "F.Cu")
@@
 	)
 	(segment
-		(start 167.576346 55.29)
-		(end 153.59 55.29)
+		(start 197.01 58.15)
+		(end 198.16 59.3)
 		(width 0.2)
 		(layer "F.Cu")
@@
 	)
 	(segment
-		(start 198.16 63.7)
-		(end 192.96 58.5)
+		(start 149.9 58.98)
+		(end 153.59 55.29)
 		(width 0.2)
 		(layer "F.Cu")
@@
 	)
 	(segment
-		(start 169.6 58.5)
-		(end 168.3 57.2)
+		(start 153.59 55.29)
+		(end 167.576346 55.29)
 		(width 0.2)
 		(layer "F.Cu")
@@
 	)
 	(segment
-		(start 171.046346 59.2)
+		(start 165.15 64.06)
 		(end 166.186346 64.06)
 		(width 0.2)
@@
 	)
 	(segment
-		(start 203.24 63.7)
-		(end 198.74 59.2)
+		(start 166.186346 64.06)
+		(end 172.496346 57.75)
 		(width 0.2)
 		(layer "B.Cu")
@@
 	)
 	(segment
-		(start 166.186346 64.06)
-		(end 165.15 64.06)
+		(start 201.69 57.75)
+		(end 203.24 59.3)
 		(width 0.2)
 		(layer "B.Cu")
@@
 	)
 	(segment
-		(start 198.74 59.2)
-		(end 171.046346 59.2)
+		(start 172.496346 57.75)
+		(end 201.69 57.75)
 		(width 0.2)
 		(layer "B.Cu")
@@
 	)
 	(segment
-		(start 190.75 102.2)
-		(end 191.35 101.6)
+		(start 163.1 74)
+		(end 163.7 74.6)
 		(width 0.2)
 		(layer "F.Cu")
@@
 	)
 	(segment
-		(start 163.1 74)
-		(end 163.7 74.6)
+		(start 175.889899 102.2)
+		(end 188.45 102.2)
 		(width 0.2)
 		(layer "F.Cu")
@@
 	)
 	(segment
-		(start 163.7 96.182944)
-		(end 165.7 96.182944)
+		(start 188.45 102.2)
+		(end 191.35 105.1)
 		(width 0.2)
 		(layer "F.Cu")
@@
 	)
 	(segment
-		(start 173.157056 103.64)
-		(end 174.449899 103.64)
+		(start 163.7 96.182944)
+		(end 165.7 96.182944)
 		(width 0.2)
 		(layer "F.Cu")
@@
 	)
 	(segment
-		(start 175.889899 102.2)
-		(end 190.75 102.2)
+		(start 173.157056 103.64)
+		(end 174.449899 103.64)
 		(width 0.2)
 		(layer "F.Cu")
@@
 	)
 	(segment
-		(start 192.65 105.3)
-		(end 191.35 106.6)
+		(start 192.65 108.8)
+		(end 191.35 110.1)
+		(width 0.2)
+		(layer "F.Cu")
+		(net 6)
+	)
+	(segment
+		(start 192.65 100.3)
+		(end 192.65 108.8)
 		(width 0.2)
 		(layer "F.Cu")
@@
 		(net 6)
 	)
-	(segment
-		(start 192.65 100.3)
-		(end 192.65 105.3)
-		(width 0.2)
-		(layer "F.Cu")
-		(net 6)
-	)
 	(via
 		(at 176.2 94.9)
@@
 	)
 	(segment
+		(start 204.35 111.6)
+		(end 205.85 110.1)
+		(width 0.2)
+		(layer "F.Cu")
+		(net 7)
+	)
+	(segment
 		(start 156.5 62)
 		(end 159.52 58.98)
@@
 	)
 	(segment
-		(start 205.85 108.6)
-		(end 202.85 111.6)
-		(width 0.2)
-		(layer "F.Cu")
-		(net 7)
-	)
-	(segment
-		(start 205.85 106.6)
-		(end 205.85 108.6)
-		(width 0.2)
-		(layer "F.Cu")
-		(net 7)
-	)
-	(segment
 		(start 151.14 87.147056)
 		(end 151.14 74.26)
@@
 	)
 	(segment
-		(start 202.85 111.6)
-		(end 175.592944 111.6)
+		(start 175.592944 111.6)
+		(end 204.35 111.6)
 		(width 0.2)
 		(layer "F.Cu")
